File: aircopter.sch (EAGLE design)
At the start: 31 parts, among them M1 WIRELESS-NRF24L01, U1 GY-521MPU6050, X1 20MHZ

Commit message: added voltage regulator
Parts:
- added C10: 2.2uF, rcl:C-USC0603
- added C11: 10uF, rcl:C-USC0603
- added IC1: STF202-22T1G, stf202_10:STF202-22T1G
- added L1: 10uH, BeagleBone_Blue_R3:INDUCTOR
Connections:
- net 3V3: now also C11.1, IC1.VOUT
- net 3V7: now also BAT.+, C10.1, C9.1, IC1.SHDN, IC1.VIN
- net GND: now also BAT.-, C10.2, C11.2, C9.2, IC1.GND
- net N$5: now also IC1.SW2, L1.1; no longer BAT.+, C9.1
- net N$6: now also IC1.SW1, L1.2; no longer BAT.-, C9.2
Other:
- note added: "Voltage Regulator"

Commit message: Add files via upload
Parts:
- C3: value 32pF -> 16pF
Changed lines of the file:
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@@
 <?xml version="1.0" encoding="utf-8"?>
 <!DOCTYPE eagle SYSTEM "eagle.dtd">
-<eagle version="9.4.0">
+<eagle version="9.7.0">
 <drawing>
 <settings>
@@
 <part name="SUPPLY2" library="Power_Symbols" library_urn="urn:adsk.eagle:library:16502351" deviceset="3V3-CIRCLE" device=""/>
 <part name="X1" library="AP_quad" deviceset="CRYSTAL" device="SMD" value="20MHZ"/>
-<part name="C3" library="rcl" library_urn="urn:adsk.eagle:library:334" deviceset="C-US" device="C0603" package3d_urn="urn:adsk.eagle:package:23616/2" value="32pF"/>
+<part name="C3" library="rcl" library_urn="urn:adsk.eagle:library:334" deviceset="C-US" device="C0603" package3d_urn="urn:adsk.eagle:package:23616/2" value="16pF"/>
 <part name="C4" library="rcl" library_urn="urn:adsk.eagle:library:334" deviceset="C-US" device="C0603" package3d_urn="urn:adsk.eagle:package:23616/2" value="32pF"/>
 <part name="GND7" library="IR_Sensor" deviceset="SUPPLY1_GND" device=""/>
